Commit message: update modelu robota

File: ros2/src/ARES_robot_model/urdf/robot.urdf.xacro (robot description, xacro)
@@ -1,4 +1,4 @@
 <?xml version="1.0"?>
-<robot name="mobile_robot" xmlns:xacro="http://www.ros.org/wiki/xacro">
+<robot name="ARES_robot_model" xmlns:xacro="http://www.ros.org/wiki/xacro">
     <!--Wymiary robota-->
     <xacro:property name="bodyWidth" value="0.4"/>
@@ -24,20 +24,30 @@
         </inertial>
     </xacro:macro>
+    <!--Meshes for robot parts-->
+    <mujoco>
+        <compiler meshdir="../meshes/" balanceinertia="false" discardvisual="false" fusestatic="false"/>
+    </mujoco>
     <!--Bryła robota-->
     <link name="body">
         <visual>
-            <origin xyz="-${bodyLength/2} 0.0 0.0" rpy="0.0 0.0 0.0"/>
+            <origin xyz="-$0.0 0.0 0.0" rpy="0.0 0.0 0.0"/>
             <geometry>
-                <box size="${bodyLength} ${bodyWidth} ${bodyHeight}"/>
+                <mesh filename="../meshes/body.STL"/>
             </geometry>
             <material name="blue"/>
         </visual>
         <collision>
-            <origin xyz="-${bodyLength/2} 0.0 0.0" rpy="0.0 0.0 0.0"/>
+            <origin xyz="-$0.0 0.0 0.0" rpy="0.0 0.0 0.0"/>
             <geometry>
                 <box size="${bodyLength} ${bodyWidth} ${bodyHeight}"/>
             </geometry>
         </collision>
-        <xacro:default_inertial mass="2.0"/>
+        <!--<collision>
+            <origin xyz="-$0.0 0.0 0.0" rpy="0.0 0.0 0.0"/>
+            <geometry>
+                <box size="${bodyLength} ${bodyWidth} ${bodyHeight}"/>
+            </geometry>
+        </collision>-->
+        <xacro:default_inertial mass="0.3"/>
     </link>
     <!--Lewe koło-->
@@ -46,5 +56,5 @@
             <origin xyz="0.0 0.0 0.0" rpy="${pi/2} 0.0 0.0"/>
             <geometry>
-                <cylinder radius="${wheelRadius}" length="0.05"/>
+                <mesh filename="../meshes/wheel.STL"/>
             </geometry>
             <material name="red"/>
@@ -53,8 +63,8 @@
             <origin xyz="0.0 0.0 0.0" rpy="${pi/2} 0.0 0.0"/>
             <geometry>
-                <cylinder radius="${wheelRadius}" length="0.05"/>
+                <cylinder radius="${wheelRadius}" length="0.02"/>
             </geometry>
         </collision>
-        <xacro:default_inertial mass="0.15"/>
+        <xacro:default_inertial mass="0.1"/>
     </link>
     <joint name="left_wheel_joint" type="continuous">
@@ -69,17 +79,17 @@
     <link name="right_wheel">
         <visual>
-            <origin xyz="0.0 0.0 0.0" rpy="${pi/2} 0.0 0.0"/>
+            <origin xyz="0.0 0.0 0.0" rpy="$-{pi/2} 0.0 0.0"/>
             <geometry>
-                <cylinder radius="${wheelRadius}" length="0.05"/>
+                <mesh filename="../meshes/wheel.STL"/>
             </geometry>
             <material name="red"/>
         </visual>
         <collision>
-            <origin xyz="0.0 0.0 0.0" rpy="${pi/2} 0.0 0.0"/>
+            <origin xyz="0.0 0.0 0.0" rpy="$-{pi/2} 0.0 0.0"/>
             <geometry>
-                <cylinder radius="${wheelRadius}" length="0.05"/>
+                <cylinder radius="${wheelRadius}" length="0.02"/>
             </geometry>
         </collision>
-        <xacro:default_inertial mass="0.15"/>
+        <xacro:default_inertial mass="0.1"/>
     </link>
     <joint name="right_wheel_joint" type="continuous">
@@ -91,26 +101,4 @@
         <dynamics damping="0.1" friction="0.1"/>
     </joint>
-    <!--Przednie koło-->
-    <link name="castor_wheel">
-        <visual>
-            <origin xyz="0.0 0.0 0.0" rpy="0.0 0.0 0.0"/>
-            <geometry>
-                <sphere radius="${castorWheelRadius}"/>
-            </geometry>
-            <material name="red"/>
-        </visual>
-        <collision>
-            <origin xyz="0.0 0.0 0.0" rpy="0.0 0.0 0.0"/>
-            <geometry>
-                <sphere radius="${castorWheelRadius}"/>
-            </geometry>
-        </collision>
-        <xacro:default_inertial mass="0.1"/>
-    </link>
-    <joint name="castor_wheel_joint" type="fixed">
-        <parent link="body"/>
-        <child link="castor_wheel"/>
-        <origin xyz="-0.05 0.0 -${bodyHeight/2}" rpy="0.0 0.0 0.0"/>
-    </joint>
     <!--LIDAR-->
     <link name="lidar">
@@ -118,5 +106,5 @@
             <origin xyz="0.0 0.0 0.0" rpy="0.0 0.0 0.0"/>
             <geometry>
-                <cylinder radius="0.1" length="0.1"/>
+                <box size="0.01 0.08 0.03"/>
             </geometry>
             <material name="green"/>
@@ -125,8 +113,8 @@
             <origin xyz="0.0 0.0 0.0" rpy="0.0 0.0 0.0"/>
             <geometry>
-                <cylinder radius="0.1" length="0.1"/>
+                <box size="0.01 0.08 0.03"/>
             </geometry>
         </collision>
-        <xacro:default_inertial mass="0.5"/>
+        <xacro:default_inertial mass="0.03"/>
     </link>
     <joint name="lidar_joint" type="fixed">
@@ -136,6 +124,6 @@
     </joint>
     <!-- Include pliku Gazebo lidar oraz differential drive controller-->
-    <xacro:include filename="$(find robot_model)/urdf/configurations.gazebo.xml"/>
-    <xacro:include filename="$(find robot_model)/urdf/lidar.gazebo.xml"/>
-    <xacro:include filename="$(find robot_model)/urdf/differential_drive.gazebo.xml"/>
+    <xacro:include filename="$(find ARES_robot_model)/urdf/configurations.gazebo.xml"/>
+    <xacro:include filename="$(find ARES_robot_model)/urdf/lidar.gazebo.xml"/>
+    <xacro:include filename="$(find ARES_robot_model)/urdf/differential_drive.gazebo.xml"/>
 </robot>

Commit message: zaktualizowano cały model robota

File: ros2/src/ARES_robot_model/urdf/robot.urdf.xacro (robot description, xacro)
@@ -2,9 +2,8 @@
 <robot name="ARES_robot_model" xmlns:xacro="http://www.ros.org/wiki/xacro">
     <!--Wymiary robota-->
-    <xacro:property name="bodyWidth" value="0.4"/>
-    <xacro:property name="bodyLength" value="0.6"/>
-    <xacro:property name="bodyHeight" value="0.2"/>
-    <xacro:property name="wheelRadius" value="0.1"/>
-    <xacro:property name="castorWheelRadius" value="0.05"/>
+    <xacro:property name="bodyWidth" value="0.09"/>
+    <xacro:property name="bodyLength" value="0.1"/>
+    <xacro:property name="bodyHeight" value="0.05"/>
+    <xacro:property name="wheelRadius" value="0.0145"/>
     <!--Kolory-->
     <material name="red">
@@ -24,29 +23,19 @@
         </inertial>
     </xacro:macro>
-    <!--Meshes for robot parts-->
-    <mujoco>
-        <compiler meshdir="../meshes/" balanceinertia="false" discardvisual="false" fusestatic="false"/>
-    </mujoco>
     <!--Bryła robota-->
     <link name="body">
         <visual>
-            <origin xyz="-$0.0 0.0 0.0" rpy="0.0 0.0 0.0"/>
+            <origin xyz="0.0 0.0 0.0" rpy="0.0 0.0 ${pi/2}"/>
             <geometry>
-                <mesh filename="../meshes/body.STL"/>
+                <mesh filename="file://$(find ARES_robot_model)/meshes/body.STL" scale="0.001 0.001 0.001"/>
             </geometry>
             <material name="blue"/>
         </visual>
         <collision>
-            <origin xyz="-$0.0 0.0 0.0" rpy="0.0 0.0 0.0"/>
+            <origin xyz="${-bodyLength/2} 0.0 ${bodyHeight/2}" rpy="0.0 0.0 ${pi/2}"/>
             <geometry>
                 <box size="${bodyLength} ${bodyWidth} ${bodyHeight}"/>
             </geometry>
         </collision>
-        <!--<collision>
-            <origin xyz="-$0.0 0.0 0.0" rpy="0.0 0.0 0.0"/>
-            <geometry>
-                <box size="${bodyLength} ${bodyWidth} ${bodyHeight}"/>
-            </geometry>
-        </collision>-->
         <xacro:default_inertial mass="0.3"/>
     </link>
@@ -54,12 +43,12 @@
     <link name="left_wheel">
         <visual>
-            <origin xyz="0.0 0.0 0.0" rpy="${pi/2} 0.0 0.0"/>
+            <origin xyz="0.0 0.01 0.0" rpy="${pi/2} 0.0 0.0"/>
             <geometry>
-                <mesh filename="../meshes/wheel.STL"/>
+                <mesh filename="file://$(find ARES_robot_model)/meshes/wheel.STL" scale="0.001 0.001 0.001"/>
             </geometry>
             <material name="red"/>
         </visual>
         <collision>
-            <origin xyz="0.0 0.0 0.0" rpy="${pi/2} 0.0 0.0"/>
+            <origin xyz="0.0 0.01 0.0" rpy="${pi/2} 0.0 0.0"/>
             <geometry>
                 <cylinder radius="${wheelRadius}" length="0.02"/>
@@ -71,5 +60,5 @@
         <parent link="body"/>
         <child link="left_wheel"/>
-        <origin xyz="-${bodyLength -0.1} ${bodyWidth/2} -${bodyHeight/2-0.05}" rpy="0.0 0.0 0.0"/>
+        <origin xyz="${0.015-bodyLength} 0.035 0.01" rpy="0.0 0.0 0.0"/>
         <axis xyz="0.0 1.0 0.0"/>
         <limit effort="100" velocity="10.0"/>
@@ -79,12 +68,12 @@
     <link name="right_wheel">
         <visual>
-            <origin xyz="0.0 0.0 0.0" rpy="$-{pi/2} 0.0 0.0"/>
+            <origin xyz="0.0 -0.01 0.0" rpy="${-pi/2} 0.0 0.0"/>
             <geometry>
-                <mesh filename="../meshes/wheel.STL"/>
+                <mesh filename="file://$(find ARES_robot_model)/meshes/wheel.STL" scale="0.001 0.001 0.001"/>
             </geometry>
             <material name="red"/>
         </visual>
         <collision>
-            <origin xyz="0.0 0.0 0.0" rpy="$-{pi/2} 0.0 0.0"/>
+            <origin xyz="0.0 -0.01 0.0" rpy="${-pi/2} 0.0 0.0"/>
             <geometry>
                 <cylinder radius="${wheelRadius}" length="0.02"/>
@@ -96,5 +85,5 @@
         <parent link="body"/>
         <child link="right_wheel"/>
-        <origin xyz="-${bodyLength -0.1} -${bodyWidth/2} -${bodyHeight/2-0.05}" rpy="0.0 0.0 0.0"/>
+        <origin xyz="${0.015-bodyLength} -0.035 0.01" rpy="0.0 0.0 0.0"/>
         <axis xyz="0.0 1.0 0.0"/>
         <limit effort="100" velocity="10.0"/>
@@ -104,14 +93,14 @@
     <link name="lidar">
         <visual>
-            <origin xyz="0.0 0.0 0.0" rpy="0.0 0.0 0.0"/>
+            <origin xyz="0.0 0.0 0.0" rpy="0.0 ${-pi/16} 0.0"/>
             <geometry>
-                <box size="0.01 0.08 0.03"/>
+                <box size="0.005 0.08 0.02"/>
             </geometry>
             <material name="green"/>
         </visual>
         <collision>
-            <origin xyz="0.0 0.0 0.0" rpy="0.0 0.0 0.0"/>
+            <origin xyz="0.0 0.0 0.0" rpy="0.0 ${-pi/16} 0.0"/>
             <geometry>
-                <box size="0.01 0.08 0.03"/>
+                <box size="0.005 0.08 0.02"/>
             </geometry>
         </collision>
@@ -121,5 +110,75 @@
         <parent link="body"/>
         <child link="lidar"/>
-        <origin xyz="-${bodyLength/2} 0.0 ${bodyHeight/2 +0.05}" rpy="0.0 0.0 0.0"/>
+        <origin xyz="-0.033 0.0 0.014" rpy="0.0 ${-pi/32} 0.0"/>
+    </joint>
+    <!--Skrzydlo lewe-->
+    <link name="left_wing">
+        <visual>
+            <origin xyz="-0.0025 0.095 0.0" rpy="0.0 0.0 0.0"/>
+            <geometry>
+                <box size="0.005 0.2 0.015"/>
+            </geometry>
+            <material name="green"/>
+        </visual>
+        <visual>
+            <origin xyz="-0.0025 0.115 -0.02" rpy="0.0 0.0 0.0"/>
+            <geometry>
+                <box size="0.005 0.16 0.025"/>
+            </geometry>
+            <material name="green"/>
+        </visual>
+        <collision>
+            <origin xyz="-0.0025 0.095 0.0" rpy="0.0 0.0 0.0"/>
+            <geometry>
+                <box size="0.005 0.2 0.015"/>
+            </geometry>
+        </collision>
+        <collision>
+            <origin xyz="-0.0025 0.115 -0.02" rpy="0.0 0.0 0.0"/>
+            <geometry>
+                <box size="0.005 0.16 0.025"/>
+            </geometry>
+        </collision>
+        <xacro:default_inertial mass="0.01"/>
+    </link>
+    <joint name="left_wing_joint" type="fixed">
+        <parent link="body"/>
+        <child link="left_wing"/>
+        <origin xyz="-0.068 0.014 0.04" rpy="0.0 0.0 0.0"/>
+    </joint>
+    <!--Skrzydlo prawo-->
+    <link name="right_wing">
+        <visual>
+            <origin xyz="-0.0025 -0.095 0.0" rpy="0.0 0.0 0.0"/>
+            <geometry>
+                <box size="0.005 0.2 0.015"/>
+            </geometry>
+            <material name="green"/>
+        </visual>
+        <visual>
+            <origin xyz="-0.0025 -0.115 -0.02" rpy="0.0 0.0 0.0"/>
+            <geometry>
+                <box size="0.005 0.16 0.025"/>
+            </geometry>
+            <material name="green"/>
+        </visual>
+        <collision>
+            <origin xyz="-0.0025 -0.095 0.0" rpy="0.0 0.0 0.0"/>
+            <geometry>
+                <box size="0.005 0.2 0.015"/>
+            </geometry>
+        </collision>
+        <collision>
+            <origin xyz="-0.0025 -0.115 -0.02" rpy="0.0 0.0 0.0"/>
+            <geometry>
+                <box size="0.005 0.16 0.025"/>
+            </geometry>
+        </collision>
+        <xacro:default_inertial mass="0.01"/>
+    </link>
+    <joint name="right_wing_joint" type="fixed">
+        <parent link="body"/>
+        <child link="right_wing"/>
+        <origin xyz="-0.068 -0.014 0.04" rpy="0.0 0.0 0.0"/>
     </joint>
     <!-- Include pliku Gazebo lidar oraz differential drive controller-->
